File: kicad_files/vga_sync_combiner_usb-c.kicad_pcb (KiCad board)
At the start: 2 copper layers, 31 x 31 mm, 19 parts, among them IC1 74HCT86, J1 VGA_RGBHV_IN, J2 POWER_SOURCE_JUMPER_HEADER, J3 JST ZR 1x2 Header, J4 RGBS_OUT_PCB_HEADER, J5 USB-C

Commit message: Add files via upload
Other:
- board text added: "VGA Sync Combiner for Audi RNS-E"
- board text removed: "VGA (RGBHV) → RGBS TTL Sync Combiner"
