File: kicad_files/vga_sync_combiner_usb-c.kicad_sch (KiCad schematic)
At the start: 37 parts, among them IC1 74HCT86, J1 VGA_RGBHV_IN, J2 POWER_SOURCE_JUMPER_HEADER, J3 JST ZR 1x2 Header, J4 RGBS_OUT_PCB_HEADER, J5 USB-C, J6 JST ZR 1x2 Cable, J7 RGBS_OUT_HOUSING (Cable), J8 REAN NYS231BG, J9 AUDI_RNS-E_32_Pin_AMP_Connect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

Commit message: Add files via upload
Other:
- note added: "VGA Sync Combiner for Audi RNS-E, 74HCT86 based"
- note removed: "VGA (RGBHV) → RGBS / C-Sync Combiner, 74HCT86 based"
- title: VGA (RGBHV) → RGBS / C-Sync Combiner, 74HCT86 based -> VGA Sync Combiner for Audi RNS-E, 74HCT86 based
Changed lines of the file:
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@@
 	(paper "A3")
 	(title_block
-		(title "VGA (RGBHV) → RGBS / C-Sync Combiner, 74HCT86 based")
+		(title "VGA Sync Combiner for Audi RNS-E, 74HCT86 based")
 		(date "2026-06-15")
 		(rev "1.0")
@@
 		)
 	)
-	(text "VGA (RGBHV) → RGBS / C-Sync Combiner, 74HCT86 based"
+	(text "VGA Sync Combiner for Audi RNS-E, 74HCT86 based"
 		(exclude_from_sim no)
-		(at 160.02 27.94 0)
+		(at 146.558 28.448 0)
 		(effects
 			(font
