File: kicad_files/vga_sync_combiner_for_audi_rns-e.kicad_sch (KiCad schematic)
At the start: 37 parts, among them IC1 74HCT86, J1 VGA_RGBHV_IN, J2 POWER_SOURCE_JUMPER_HEADER, J3 JST ZR 1x2 Header, J4 RGBS_OUT_PCB_HEADER, J5 USB-C, J6 JST ZR 1x2 Cable, J7 RGBS_OUT_HOUSING (Cable), J8 REAN NYS231BG, J9 AUDI_RNS-E_32_Pin_AMP_Connect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

Commit message: Add files via upload
Parts:
- C1, C2, C3, C4, D1, IC1, J1, J2, J3, J4, J5, JMP1, R1, R2, R3, R4, R5, R6: Category (none) -> PCB
- CBL1, CBL2, CP1, CP10, CP11, CP12, CP2, CP3, CP4, CP5, CP7, CP8, CP9, J6, J7, J8, J9: Category (none) -> Cable
- H1, H2: now in the parts list

Commit message: Add files via upload
Parts:
- H1, H2: Category (none) -> PCB; now left out of the parts list
- JMP1: Category PCB -> Accessory
Changed lines of the file:
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@@
 			)
 		)
-		(property "Description" "Generic connector, single row, 01x02, script generated (kicad-library-utils/schlib/autogen/connector/)"
+		(property "Description" "JST ZR 2-pin cable assembly for optional external 5V input. Excluded from board, included in complete BOM. PCB polarity: Pin 2 = +5V, Pin 1 = GND."
 			(at 116.84 134.62 0)
 			(hide yes)
@@
 			)
 		)
-		(property "Description" "Generic connector, single row, 01x05, script generated (kicad-library-utils/schlib/autogen/connector/)"
+		(property "Description" "TE Micro-MATE-N-LOK 5-position cable housing for RGBS output cable. Excluded from board, included in complete BOM."
 			(at 41.91 232.41 0)
 			(hide yes)
@@
 			)
 		)
-		(property "Description" "Generic connector, double row, 02x16, top/bottom pin numbering scheme (row 1: 1...pins_per_row, row2: pins_per_row+1 ... num_pins), script generated (kicad-library-utils/schlib/autogen/connector/)"
+		(property "Description" "Audi/VW 32-pin RNS-E AV connector housing for RGBS/audio cable connection. Excluded from board, included in complete BOM."
 			(at 182.88 247.65 0)
 			(hide yes)
@@
 			)
 		)
-		(property "Category" "PCB"
+		(property "Category" "Accessory"
 			(at 83.82 116.84 0)
 			(hide yes)
@@
 		(body_style 1)
 		(exclude_from_sim no)
-		(in_bom yes)
+		(in_bom no)
 		(on_board yes)
 		(in_pos_files yes)
@@
 			)
 		)
-		(property "Category" ""
+		(property "Category" "PCB"
 			(at 43.18 104.14 90)
 			(hide yes)
@@
 			)
 		)
-		(property "Description" "Generic connector, double row, 02x03, odd/even pin numbering scheme (row 1 odd numbers, row 2 even numbers), script generated (kicad-library-utils/schlib/autogen/connector/)"
+		(property "Description" "Shielded stereo audio cable, Cordial CPK 220 BK. Carries left/right audio and ground to the 3.5mm TRS plug."
 			(at 93.98 257.81 0)
 			(hide yes)
@@
 			)
 		)
-		(property "Description" "Generic connector, double row, 02x06, odd/even pin numbering scheme (row 1 odd numbers, row 2 even numbers), script generated (kicad-library-utils/schlib/autogen/connector/)"
+		(property "Description" "Shielded RGBS cable, LAPP UNITRONIC LiYCY 5x0.34mm², black. Carries R, G, B, C-Sync and GND to the Audi RNS-E connector."
 			(at 93.98 232.41 0)
 			(hide yes)
@@
 		(body_style 1)
 		(exclude_from_sim no)
-		(in_bom yes)
+		(in_bom no)
 		(on_board yes)
 		(in_pos_files yes)
@@
 			)
 		)
-		(property "Category" ""
+		(property "Category" "PCB"
 			(at 43.18 110.49 90)
 			(hide yes)
